Commit message: updates to 3d mapping

File: description/depth_camera.xacro (robot description, xacro)
@@ -34,6 +34,6 @@
                 </image>
                 <clip>
-                    <near>0.05</near>
-                    <far>8.0</far>
+                    <near>0.2</near>
+                    <far>10.0</far>
                 </clip>
             </camera>

File: description/gazebo_control.xacro (robot description, xacro)
@@ -18,4 +18,5 @@
             <!-- Output -->
             <odometry_frame>odom</odometry_frame>
+            <odometry_topic>odom</odometry_topic>
             <robot_base_frame>base_link</robot_base_frame>
             <publish_odom>true</publish_odom>

File: description/robot.urdf.xacro (robot description, xacro)
@@ -1,5 +1,5 @@
 <?xml version="1.0"?>
 <robot xmlns:xacro="http://www.ros.org/wiki/xacro"  name="robot">
-    <xacro:arg name="use_ros2_control" default="true" />
+    <xacro:arg name="use_ros2_control" default="false" />
     <xacro:include filename="robot_core.xacro" />
     <xacro:if value="$(arg use_ros2_control)">

File: description/robot_core.xacro (robot description, xacro)
@@ -24,5 +24,5 @@
         <parent link="base_link"/>
         <child link="base_footprint"/>
-        <origin xyz= "0 0 0" rpy= "0 0 0"/>
+        <origin xyz= "0 0 -0.05" rpy= "0 0 0"/>
     </joint>
     <link name= "base_footprint">
