Commit message: adjusted lidar xacro

File: description/lidar.xacro (robot description, xacro)
@@ -4,8 +4,10 @@
         <parent link="chassis"/>
         <child link="laser_frame"/>
-        <origin xyz="0.172 0 0.068" rpy="0 0 0"/>
+        <origin xyz="0.172 0 0.085" rpy="0 0 0"/>
+        <!-- the rplidar c1 has it laser scans emmitted at a height of 29.8mm from the base od the sensor, this was added to the height of the chasis to get 85mm used above -->
     </joint>
     <link name="laser_frame">
         <visual>
+            <origin xyz="0 0 -0.017"/>
             <geometry>
                 <box size="0.055 0.055 0.023"/>
@@ -14,5 +16,5 @@
         </visual>
         <visual>
-            <origin xyz="0 0 0.021"/>
+            <origin xyz="0 0 0.003"/>
             <geometry>
                 <cylinder radius="0.022" length="0.018"/>
@@ -22,8 +24,8 @@
         <collision>
             <geometry>
-                <cylinder radius="0.05" length="0.04"/>
+                <cylinder radius="0.022" length="0.018"/>
             </geometry>
         </collision>
-        <xacro:inertial_cylinder mass="0.1" length="0.04" radius="0.05">
+        <xacro:inertial_cylinder mass="0.1" length="0.018" radius="022">
             <origin xyz="0 0 0" rpy="0 0 0"/>
         </xacro:inertial_cylinder>

File: description/robot.urdf.xacro (robot description, xacro)
@@ -11,5 +11,5 @@
     </xacro:unless>
     <xacro:include filename="lidar.xacro" />
-    <!-- <xacro:include filename="camera.xacro" /> -->
+    <xacro:include filename="camera.xacro" />
     <!-- <xacro:include filename="depth_camera.xacro" /> -->
    <!-- <xacro:include filename="face.xacro" /> -->
