Commit message: fixed teleop and camera display in rviz

File: description/camera.xacro (robot description, xacro)
@@ -46,5 +46,5 @@
                 </clip>
             </camera>
-            <topic>camara/image_raw</topic>
+            <topic>camera/image_raw</topic>
             <gz_frame_id>camera_link_optical</gz_frame_id>
         </sensor>

File: description/lidar.xacro (robot description, xacro)
@@ -27,6 +27,6 @@
             </geometry>
         </collision>
-        <xacro:inertial_cylinder mass="0.1" length="0.018" radius="022">
-            <origin xyz="0 0 0" rpy="0 0 0"/>
+        <xacro:inertial_cylinder mass="0.1" length="0.018" radius="0.022">
+            <origin xyz="0 0 0.003" rpy="0 0 0"/>
         </xacro:inertial_cylinder>
     </link>

File: description/robot_core.xacro (robot description, xacro)
@@ -38,5 +38,5 @@
         <parent link="base_link"/>
         <child link="base_footprint"/>
-        <origin xyz= "0 0 -0.05" rpy= "0 0 0"/>
+        <origin xyz= "0 0 0.057" rpy= "0 0 0"/>
     </joint>
     <link name= "base_footprint">
@@ -44,5 +44,5 @@
     <!-- CHASSIS LINK -->
     <joint name="chassis_joint" type="fixed">
-        <parent link="base_link"/>
+        <parent link="base_footprint"/>
         <child link="chassis"/>
         <origin xyz="-0.116 0 0"/>
@@ -71,5 +71,5 @@
     <!-- rear LEFT WHEEL LINK -->
     <joint name="left_wheel_joint" type="continuous">
-        <parent link="base_link"/>
+        <parent link="base_footprint"/>
         <child link="left_wheel"/>
         <origin xyz="-0.084 0.101 -0.024" rpy="-${pi/2} 0 0" />
@@ -85,5 +85,5 @@
         <collision>
             <geometry>
-                <sphere radius="0.065" />
+                <sphere radius="0.0325" />
             </geometry>
         </collision>
@@ -97,8 +97,8 @@
     <!-- rear RIGHT WHEEL LINK -->
     <joint name="right_wheel_joint" type="continuous">
-        <parent link="base_link"/>
+        <parent link="base_footprint"/>
         <child link="right_wheel"/>
-        <origin xyz="-0.084 -0.101 -0.024" rpy="-${pi/2} 0 0" />
-        <axis xyz="0 0 1"/>
+        <origin xyz="-0.084 -0.101 -0.024" rpy="${pi/2} 0 0" />
+        <axis xyz="0 0 -1"/>
     </joint>
     <link name="right_wheel">
@@ -111,5 +111,5 @@
         <collision>
             <geometry>
-                <sphere radius="0.065" />
+                <sphere radius="0.0325" />
             </geometry>
         </collision>
@@ -145,5 +145,5 @@
  <!-- front LEFT WHEEL LINK -->
     <joint name="front_left_wheel_joint" type="continuous">
-        <parent link="base_link"/>
+        <parent link="base_footprint"/>
         <child link="front_left_wheel"/>
         <origin xyz="0.084 0.101 -0.024" rpy="-${pi/2} 0 0" />
@@ -159,5 +159,5 @@
         <collision>
             <geometry>
-                <sphere radius="0.065" />
+                <sphere radius="0.0325" />
             </geometry>
         </collision>
@@ -171,19 +171,19 @@
     <!-- front RIGHT WHEEL LINK -->
     <joint name="front_right_wheel_joint" type="continuous">
-        <parent link="base_link"/>
+        <parent link="base_footprint"/>
         <child link="front_right_wheel"/>
-        <origin xyz="0.084 -0.101 -0.024" rpy="-${pi/2} 0 0" />
-        <axis xyz="0 0 1"/>
+        <origin xyz="0.084 -0.101 -0.024" rpy="${pi/2} 0 0" />
+        <axis xyz="0 0 -1"/>
     </joint>
     <link name="front_right_wheel">
         <visual>
             <geometry>
-                <cylinder radius="0.025" length="0.027"/>
-            </geometry>
-            <material name="blue"/>
-        </visual>
-        <collision>
-            <geometry>
-                <sphere radius="0.065" />
+                <cylinder radius="0.0325" length="0.027"/>
+            </geometry>
+            <material name="blue"/>
+        </visual>
+        <collision>
+            <geometry>
+                <sphere radius="0.0325" />
             </geometry>
         </collision>
