Commit message: coverted to a 4W-DiffDrive

File: description/gazebo_control.xacro (robot description, xacro)
@@ -4,7 +4,12 @@
         <plugin name="diff_drive" filename="libgazebo_ros_diff_drive.so">
             <!-- Wheel Information -->
+            <num_wheel_pairs>2</num_wheel_pairs>
             <left_joint>left_wheel_joint</left_joint>
             <right_joint>right_wheel_joint</right_joint>
+            <left_joint>front_left_wheel_joint</left_joint>
+            <right_joint>front_right_wheel_joint</right_joint>
             <wheel_separation>0.35</wheel_separation>
+            <wheel_separation>0.35</wheel_separation>
+            <wheel_diameter>0.1</wheel_diameter>
             <wheel_diameter>0.1</wheel_diameter>
             <!-- Limits -->

File: description/robot_core.xacro (robot description, xacro)
@@ -55,9 +55,9 @@
         <material>Gazebo/White</material>
     </gazebo>
-    <!-- LEFT WHEEL LINK -->
+    <!-- rear LEFT WHEEL LINK -->
     <joint name="left_wheel_joint" type="continuous">
         <parent link="base_link"/>
         <child link="left_wheel"/>
-        <origin xyz="0.0 0.175 0" rpy="-${pi/2} 0 0" />
+        <origin xyz="-0.04 0.175 0" rpy="-${pi/2} 0 0" />
         <axis xyz="0 0 1"/>
     </joint>
@@ -81,9 +81,9 @@
         <material>Gazebo/Blue</material>
     </gazebo>
-    <!-- RIGHT WHEEL LINK -->
+    <!-- rear RIGHT WHEEL LINK -->
     <joint name="right_wheel_joint" type="continuous">
         <parent link="base_link"/>
         <child link="right_wheel"/>
-        <origin xyz="0 -0.175 0" rpy="${pi/2} 0 0" />
+        <origin xyz="-0.04 -0.175 0" rpy="${pi/2} 0 0" />
         <axis xyz="0 0 -1"/>
     </joint>
@@ -107,5 +107,5 @@
         <material>Gazebo/Blue</material>
     </gazebo>
-    <!-- CASTER WHEEL LINK -->
+    <!-- CASTER WHEEL LINK
     <joint name="caster_wheel_joint" type="fixed">
         <parent link="chassis"/>
@@ -128,5 +128,57 @@
             <origin xyz="0 0 0" rpy="0 0 0"/>
         </xacro:inertial_sphere>
+    </link> -->
+ <!-- front LEFT WHEEL LINK -->
+    <joint name="front_left_wheel_joint" type="continuous">
+        <parent link="base_link"/>
+        <child link="front_left_wheel"/>
+        <origin xyz="0.14 0.175 0" rpy="-${pi/2} 0 0" />
+        <axis xyz="0 0 1"/>
+    </joint>
+    <link name="front_left_wheel">
+        <visual>
+            <geometry>
+                <cylinder radius="0.05" length="0.04"/>
+            </geometry>
+            <material name="blue"/>
+        </visual>
+        <collision>
+            <geometry>
+                <sphere radius="0.05" />
+            </geometry>
+        </collision>
+        <xacro:inertial_cylinder mass="0.1" length="0.04" radius="0.05">
+            <origin xyz="0 0 0" rpy="0 0 0"/>
+        </xacro:inertial_cylinder>
     </link>
+    <gazebo reference="front_left_wheel">
+        <material>Gazebo/Blue</material>
+    </gazebo>
+    <!-- front RIGHT WHEEL LINK -->
+    <joint name="front_right_wheel_joint" type="continuous">
+        <parent link="base_link"/>
+        <child link="front_right_wheel"/>
+        <origin xyz="0.14 -0.175 0" rpy="${pi/2} 0 0" />
+        <axis xyz="0 0 -1"/>
+    </joint>
+    <link name="front_right_wheel">
+        <visual>
+            <geometry>
+                <cylinder radius="0.05" length="0.04"/>
+            </geometry>
+            <material name="blue"/>
+        </visual>
+        <collision>
+            <geometry>
+                <sphere radius="0.05" />
+            </geometry>
+        </collision>
+        <xacro:inertial_cylinder mass="0.1" length="0.04" radius="0.05">
+            <origin xyz="0 0 0" rpy="0 0 0"/>
+        </xacro:inertial_cylinder>
+    </link>
+    <gazebo reference="front_right_wheel">
+        <material>Gazebo/Blue</material>
+    </gazebo>
     <gazebo reference="caster_wheel">
         <material>Gazebo/Black</material>

Commit message: resolved all errors on terminal when runnung gazebo

File: description/gazebo_control.xacro (robot description, xacro)
@@ -9,11 +9,9 @@
             <left_joint>front_left_wheel_joint</left_joint>
             <right_joint>front_right_wheel_joint</right_joint>
-            <wheel_separation>0.35</wheel_separation>
-            <wheel_separation>0.35</wheel_separation>
-            <wheel_radius>0.1</wheel_radius>
-            <wheel_radius>0.1</wheel_radius>
-            <left_joint>left_wheel_joint</left_joint>
-            <right_joint>right_wheel_joint</right_joint>
-            <wheel_separation>0.297</wheel_separation>
+            <wheel_separation>0.168</wheel_separation>
+            <wheel_separation>0.168</wheel_separation>
+            <wheel_radius>0.0325</wheel_radius>
+            <wheel_radius>0.0325</wheel_radius>
+            <!-- <wheel_separation>0.297</wheel_separation> -->
             <!--<wheel_radius>0.033</wheel_radius> -->
             <!-- Limits -->
@@ -34,4 +32,6 @@
             <joint_name>left_wheel_joint</joint_name>
             <joint_name>right_wheel_joint</joint_name>
+            <joint_name>front_left_wheel_joint</joint_name>
+            <joint_name>front_right_wheel_joint</joint_name>
         </plugin>
     </gazebo>

File: description/robot_core.xacro (robot description, xacro)
@@ -195,8 +195,8 @@
         <material>Gazebo/Blue</material>
     </gazebo>
-    <gazebo reference="caster_wheel">
+    <!-- <gazebo reference="caster_wheel">
         <material>Gazebo/Black</material>
         <mu1 value="0.001"/>
         <mu2 value="0.001"/>
-    </gazebo>
+    </gazebo> -->
 </robot>

File: description/ros2_control.xacro (robot description, xacro)
@@ -52,4 +52,20 @@
                 <state_interface name="position"/>
             </joint>
+            <joint name="front_left_wheel_joint">
+                <command_interface name="velocity">
+                    <param name="min">-10</param>
+                    <param name="max">10</param>
+                </command_interface>
+                <state_interface name="velocity"/>
+                <state_interface name="position"/>
+            </joint>
+            <joint name="front_right_wheel_joint">
+                <command_interface name="velocity">
+                    <param name="min">-10</param>
+                    <param name="max">10</param>
+                </command_interface>
+                <state_interface name="velocity"/>
+                <state_interface name="position"/>
+            </joint>
         </ros2_control>
     </xacro:if>

Commit message: gz_bridge,  modified robot urdf

File: description/gazebo_control.xacro (robot description, xacro)
@@ -9,6 +9,6 @@
             <left_joint>front_left_wheel_joint</left_joint>
             <right_joint>front_right_wheel_joint</right_joint>
-            <wheel_separation>0.168</wheel_separation>
-            <wheel_separation>0.168</wheel_separation>
+            <wheel_separation>0.202</wheel_separation>
+            <wheel_separation>0.202</wheel_separation>
             <wheel_radius>0.0325</wheel_radius>
             <wheel_radius>0.0325</wheel_radius>

File: description/robot_core.xacro (robot description, xacro)
@@ -38,5 +38,5 @@
         <parent link="base_link"/>
         <child link="base_footprint"/>
-        <origin xyz= "0 0 0.057" rpy= "0 0 0"/>
+        <origin xyz= "0 0 0" rpy= "0 0 0"/>
     </joint>
     <link name= "base_footprint">
@@ -44,7 +44,7 @@
     <!-- CHASSIS LINK -->
     <joint name="chassis_joint" type="fixed">
-        <parent link="base_footprint"/>
+        <parent link="base_link"/>
         <child link="chassis"/>
-        <origin xyz="-0.116 0 0"/>
+        <origin xyz="-0.116 0 0.057"/>
     </joint>
     <link name="chassis">
@@ -71,7 +71,7 @@
     <!-- rear LEFT WHEEL LINK -->
     <joint name="left_wheel_joint" type="continuous">
-        <parent link="base_footprint"/>
+        <parent link="base_link"/>
         <child link="left_wheel"/>
-        <origin xyz="-0.084 0.101 -0.024" rpy="-${pi/2} 0 0" />
+        <origin xyz="-0.084 0.101 0.0325" rpy="-${pi/2} 0 0" />
         <axis xyz="0 0 1"/>
     </joint>
@@ -97,7 +97,7 @@
     <!-- rear RIGHT WHEEL LINK -->
     <joint name="right_wheel_joint" type="continuous">
-        <parent link="base_footprint"/>
+        <parent link="base_link"/>
         <child link="right_wheel"/>
-        <origin xyz="-0.084 -0.101 -0.024" rpy="${pi/2} 0 0" />
+        <origin xyz="-0.084 -0.101 0.0325" rpy="${pi/2} 0 0" />
         <axis xyz="0 0 -1"/>
     </joint>
@@ -145,7 +145,7 @@
  <!-- front LEFT WHEEL LINK -->
     <joint name="front_left_wheel_joint" type="continuous">
-        <parent link="base_footprint"/>
+        <parent link="base_link"/>
         <child link="front_left_wheel"/>
-        <origin xyz="0.084 0.101 -0.024" rpy="-${pi/2} 0 0" />
+        <origin xyz="0.084 0.101 0.0325" rpy="-${pi/2} 0 0" />
         <axis xyz="0 0 1"/>
     </joint>
@@ -171,7 +171,7 @@
     <!-- front RIGHT WHEEL LINK -->
     <joint name="front_right_wheel_joint" type="continuous">
-        <parent link="base_footprint"/>
+        <parent link="base_link"/>
         <child link="front_right_wheel"/>
-        <origin xyz="0.084 -0.101 -0.024" rpy="${pi/2} 0 0" />
+        <origin xyz="0.084 -0.101 0.0325" rpy="${pi/2} 0 0" />
         <axis xyz="0 0 -1"/>
     </joint>

File: description/ros2_control.xacro (robot description, xacro)
@@ -1,3 +1,104 @@
 <?xml version="1.0"?>
+<robot xmlns:xacro="http://www.ros.org/wiki/xacro">
+    <xacro:macro name="tetris" params="name"/>
+    <xacro:unless value="$(arg sim_mode)">
+        <ros2_control name="${name}_front" type="system">
+            <hardware>
+                <plugin>epmc_ros_hw_plugin/EPMCHardwareInterface</plugin>
+                <param name="motorA_wheel_name">front_left_wheel_joint</param>
+                <param name="motorB_wheel_name">front_right_wheel_joint</param>
+                <param name="port">/dev/serial/by-path/pci-0000:00:14.0-usb-0:1.2:1.0-port0</param>
+                <param name="cmd_vel_timeout_ms">2000</param>
+            </hardware>
+            <joint name="front_left_wheel_joint">
+                <command_interface name="velocity">
+                    <param name="min">-10.0</param>
+                    <param name="max">10.0</param>
+                </command_interface>
+                <state_interface name="position"/>
+                <state_interface name="velocity"/>
+            </joint>
+            <joint name="front_right_wheel_joint">
+                <command_interface name="velocity">
+                    <param name="min">-10.0</param>
+                    <param name="max">10.0</param>
+                </command_interface>
+                <state_interface name="position"/>
+                <state_interface name="velocity"/>
+            </joint>
+        </ros2_control>
+        <ros2_control name="${name}_rear" type="system">
+            <hardware>
+                <plugin>epmc_ros_hw_plugin/EPMCHardwareInterface</plugin>
+                <param name="motorA_wheel_name">rear_left_wheel_joint</param>
+                <param name="motorB_wheel_name">rear_right_wheel_joint</param>
+                <param name="port">/dev/serial/by-path/pci-0000:00:14.0-usb-0:1.1:1.0-port0</param>
+                <param name="cmd_vel_timeout_ms">2000</param>
+            </hardware>
+            <joint name="rear_left_wheel_joint">
+                <command_interface name="velocity">
+                    <param name="min">-10.0</param>
+                    <param name="max">10.0</param>
+                </command_interface>
+                <state_interface name="position"/>
+                <state_interface name="velocity"/>
+            </joint>
+            <joint name="rear_right_wheel_joint">
+                <command_interface name="velocity">
+                    <param name="min">-10.0</param>
+                    <param name="max">10.0</param>
+                </command_interface>
+                <state_interface name="position"/>
+                <state_interface name="velocity"/>
+            </joint>
+        </ros2_control>
+    </xacro:unless>
+    <xacro:if value="$(arg sim_mode)">
+        <ros2_control name="GazeboSystem" type="system">
+            <hardware>
+                <plugin>gz_ros2_control/GazeboSimSystem</plugin>
+            </hardware>
+            <joint name="left_wheel_joint">
+                <command_interface name="velocity">
+                    <param name="min">-10</param>
+                    <param name="max">10</param>
+                </command_interface>
+                <state_interface name="velocity"/>
+                <state_interface name="position"/>
+            </joint>
+            <joint name="right_wheel_joint">
+                <command_interface name="velocity">
+                    <param name="min">-10</param>
+                    <param name="max">10</param>
+                </command_interface>
+                <state_interface name="velocity"/>
+                <state_interface name="position"/>
+            </joint>
+            <joint name="front_left_wheel_joint">
+                <command_interface name="velocity">
+                    <param name="min">-10</param>
+                    <param name="max">10</param>
+                </command_interface>
+                <state_interface name="velocity"/>
+                <state_interface name="position"/>
+            </joint>
+            <joint name="front_right_wheel_joint">
+                <command_interface name="velocity">
+                    <param name="min">-10</param>
+                    <param name="max">10</param>
+                </command_interface>
+                <state_interface name="velocity"/>
+                <state_interface name="position"/>
+            </joint>
+        </ros2_control>
+    </xacro:if>
+    <gazebo>
+        <plugin name="gz_ros2_control::GazeboSimROS2ControlPlugin" filename="libgz_ros2_control-system.so">
+            <parameters>$(find articubot_one)/config/my_controllers.yaml</parameters>
+            <parameters>$(find articubot_one)/config/gaz_ros2_ctl_use_sim.yaml</parameters>
+        </plugin>
+    </gazebo>
+</robot>
+<!-- <?xml version="1.0"?>
 <robot xmlns:xacro="http://www.ros.org/wiki/xacro">
     <xacro:unless value="$(arg sim_mode)">
@@ -76,3 +177,3 @@
         </plugin>
     </gazebo>
-</robot>
+</robot> -->
